Commit message: Driver working and enforcing limits

File: motor_controller/urdf/lysander.xacro (robot description, xacro)
@@ -1,14 +1,14 @@
 <?xml version="1.0"?>
 <robot xmlns:xacro="http://www.ros.org/wiki/xacro" name="lysander">
-  <xacro:property name="body_length" value="0.6096" />>
-  <xacro:property name="body_width" value="0.3048" />
+  <xacro:property name="body_length" value="0.3048" />>
+  <xacro:property name="body_width" value="0.2286" />
   <xacro:property name="wheel_forward_of_center_distance" value=".0762" />>
-  <xacro:property name="wheel_radius" value="0.0762" />
+  <xacro:property name="wheel_radius" value="0.376991118430775" />
   <xacro:property name="wheel_spacer" value="0.00635" />>
-  <xacro:property name="wheel_width" value="0.040" />
+  <xacro:property name="wheel_width" value="0.060" />
   <!--xacro:include filename="$(find m1)/robots/m1.gazebo" /-->
   <gazebo>
     <plugin name="gazebo_ros_control" filename="libgazebo_ros_control.so">
-      <robotNamespace>/lysander</robotNamespace>
+      <!--robotNamespace>/lysander</robotNamespace-->
       <robotSimType>gazebo_ros_control/DefaultRobotHWSim</robotSimType>
     </plugin>
@@ -55,4 +55,9 @@
           izz="1.0" />
     </inertial>
+    <collision name="lwheel_collision">
+      <geometry>
+        <cylinder length="${wheel_width}" radius="${wheel_radius}" />
+      </geometry>
+    </collision>
   </link>
   <joint name="base_to_lwheel" type="continuous">
@@ -61,4 +66,5 @@
     <origin xyz="${wheel_forward_of_center_distance} ${(body_width/2)+wheel_spacer+wheel_width} ${wheel_radius}" rpy="1.5708 0 0"/>
     <axis xyz="0 0 1" />
+    <limit effort="0.0"  velocity="0.75" />
   </joint>
   <transmission name="left_wheel">
@@ -88,4 +94,9 @@
           izz="1.0" />
     </inertial>
+    <collision name="rwheel_collision">
+      <geometry>
+        <cylinder length="${wheel_width}" radius="${wheel_radius}" />
+      </geometry>
+    </collision>
   </link>
   <joint name="base_to_rwheel" type="continuous">
@@ -94,4 +105,5 @@
     <origin xyz="${wheel_forward_of_center_distance} -${(body_width/2)+wheel_spacer+wheel_width} ${wheel_radius}" rpy="-1.5708 0 0"/>
     <axis xyz="0 0 1" />
+    <limit effort="0.0"  velocity="0.75" />
   </joint>
   <transmission name="right_wheel">

Commit message: Better URDF model positions

File: motor_controller/urdf/lysander.xacro (robot description, xacro)
@@ -1,10 +1,19 @@
 <?xml version="1.0"?>
 <robot xmlns:xacro="http://www.ros.org/wiki/xacro" name="lysander">
-  <xacro:property name="body_length" value="0.3048" />>
+  <xacro:property name="body_length" value="0.3048" />
   <xacro:property name="body_width" value="0.2286" />
-  <xacro:property name="wheel_forward_of_center_distance" value=".0762" />>
-  <xacro:property name="wheel_radius" value="0.376991118430775" />
-  <xacro:property name="wheel_spacer" value="0.00635" />>
+  <xacro:property name="body_height" value="0.0508" />
+  <xacro:property name="fwheel_offset" value="-0.13" />
+  <xacro:property name="motor_height" value="0.0254" />
+  <xacro:property name="scanner_height" value="0.015" />
+  <xacro:property name="scanner_length" value="0.045" />
+  <xacro:property name="scanner_width" value="0.015" />
+  <xacro:property name="wheel_forward_of_center_distance" value=".0762" />
+  <xacro:property name="wheel_radius" value="0.06" />
+  <xacro:property name="wheel_spacer" value="0.00254" />
   <xacro:property name="wheel_width" value="0.060" />
+  <xacro:property name="body_center_height" value="${wheel_radius+(motor_height/2)+(body_height/2)}" />
+  <xacro:property name="scanner_x_offset" value="${(body_length/2)-(scanner_width/2)}" />
+  <xacro:property name="scanner_z_offset" value="${body_center_height+(body_height/2)+(scanner_height/2)+.00508}" />
   <!--xacro:include filename="$(find m1)/robots/m1.gazebo" /-->
   <gazebo>
@@ -25,7 +34,7 @@
     <visual>
       <geometry>
-        <box size="${body_length} ${body_width} 0.12"/>
+        <box size="${body_length} ${body_width} 0.0508"/>
       </geometry>
-      <origin rpy="0 0 0" xyz="0 0 0.085"/>
+      <origin rpy="0 0 0" xyz="0 0 ${body_center_height}"/>
       <material name="base" />
     </visual>
@@ -64,5 +73,5 @@
     <parent link="base_link"/>
     <child link="lwheel"/>
-    <origin xyz="${wheel_forward_of_center_distance} ${(body_width/2)+wheel_spacer+wheel_width} ${wheel_radius}" rpy="1.5708 0 0"/>
+    <origin xyz="${wheel_forward_of_center_distance} ${(body_width/2)+wheel_spacer+(wheel_width/2)} ${wheel_width}" rpy="1.5708 0 0"/>
     <axis xyz="0 0 1" />
     <limit effort="0.0"  velocity="0.75" />
@@ -103,5 +112,5 @@
     <parent link="base_link"/>
     <child link="rwheel"/>
-    <origin xyz="${wheel_forward_of_center_distance} -${(body_width/2)+wheel_spacer+wheel_width} ${wheel_radius}" rpy="-1.5708 0 0"/>
+    <origin xyz="${wheel_forward_of_center_distance} -${(body_width/2)+wheel_spacer+(wheel_width/2)} ${wheel_width}" rpy="-1.5708 0 0"/>
     <axis xyz="0 0 1" />
     <limit effort="0.0"  velocity="0.75" />
@@ -122,5 +131,5 @@
         <cylinder length="0.060" radius="0.023"/>
       </geometry>
-      <origin rpy="0 0 0" xyz="0.13 0 0.08"/>
+      <origin rpy="0 0 0" xyz="${fwheel_offset} 0 0.08"/>
       <material name="white">
         <color rgba="0.3 0.4 0.5 1"/>
@@ -161,5 +170,5 @@
     <parent link="base_link"/>
     <child link="fwheel"/>
-    <origin xyz="0.13 0 0.02" rpy="0 0 0"/>
+    <origin xyz="${fwheel_offset} 0 0.02" rpy="0 0 0"/>
     <axis xyz="0 0 1" />
   </joint>
@@ -167,7 +176,7 @@
     <visual>
       <geometry>
-        <box size="0.015 0.045 0.015"/>
+        <box size="${scanner_width} ${scanner_length} ${scanner_height}"/>
       </geometry>
-      <origin rpy="0 0 0" xyz="0.022 0 0.015"/>
+      <origin rpy="0 0 0" xyz="0 0 0"/>
       <material name="black">
         <color rgba="0.5 0 0 1"/>
@@ -186,5 +195,5 @@
     <parent link="base_link"/>
     <child link="scanner"/>
-    <origin xyz="0.105 0 0.22" rpy="0 0 0"/>
+    <origin xyz="${scanner_x_offset} 0  ${scanner_z_offset}" rpy="0 0 0"/>
   </joint>
 </robot>

Commit message: Basic gazebo working

File: motor_controller/urdf/lysander.xacro (robot description, xacro)
@@ -19,6 +19,6 @@
   <gazebo>
     <plugin name="gazebo_ros_control" filename="libgazebo_ros_control.so">
-      <!--robotNamespace>/lysander</robotNamespace-->
       <robotSimType>gazebo_ros_control/DefaultRobotHWSim</robotSimType>
+      <legacyModeNS>true</legacyModeNS>
     </plugin>
   </gazebo>
@@ -30,4 +30,9 @@
     <color rgba="0.6 0.5 0.5 1" />
   </material>
+  <link name="world" />
+  <joint name="fixed" type="fixed" >
+    <parent link="world" />
+    <child link="base_link" />
+  </joint>
   <!-- Parts -->
   <link name="base_link">

Commit message: First try at LysanderMotor.cpp

File: motor_controller/urdf/lysander.xacro (robot description, xacro)
@@ -1,13 +1,14 @@
 <?xml version="1.0"?>
-<robot xmlns:xacro="http://www.ros.org/wiki/xacro" name="lysander">
+<robot xmlns:xacro="http://ros.org/wiki/xacro" name="lysander">
+  <xacro:include filename="$(find motor_controller)/urdf/wheel.urdf.xacro" />
+  <xacro:property name="body_height" value="0.0508" />
   <xacro:property name="body_length" value="0.3048" />
   <xacro:property name="body_width" value="0.2286" />
-  <xacro:property name="body_height" value="0.0508" />
   <xacro:property name="fwheel_offset" value="-0.13" />
+  <xacro:property name="wheel_forward_of_center_distance" value=".0762" />
   <xacro:property name="motor_height" value="0.0254" />
   <xacro:property name="scanner_height" value="0.015" />
   <xacro:property name="scanner_length" value="0.045" />
   <xacro:property name="scanner_width" value="0.015" />
-  <xacro:property name="wheel_forward_of_center_distance" value=".0762" />
   <xacro:property name="wheel_radius" value="0.06" />
   <xacro:property name="wheel_spacer" value="0.00254" />
@@ -16,4 +17,10 @@
   <xacro:property name="scanner_x_offset" value="${(body_length/2)-(scanner_width/2)}" />
   <xacro:property name="scanner_z_offset" value="${body_center_height+(body_height/2)+(scanner_height/2)+.00508}" />
+  <material name="base">
+    <color rgba="0.25 0.25 0.53 1" />>
+  </material>
+  <material name="wheel">
+    <color rgba="0.6 0.5 0.5 1" />
+  </material>
   <!--xacro:include filename="$(find m1)/robots/m1.gazebo" /-->
   <gazebo>
@@ -23,24 +30,48 @@
     </plugin>
   </gazebo>
-  <!-- Materials -->
-  <material name="base">
-    <color rgba="0.0 0.25 0.53 1" />>
-  </material>
-  <material name="wheel">
-    <color rgba="0.6 0.5 0.5 1" />
-  </material>
-  <link name="world" />
-  <joint name="fixed" type="fixed" >
-    <parent link="world" />
-    <child link="base_link" />
+  <!-- Base footprint is on the ground under the robot -->
+  <link name="base_footprint"/>
+  <joint name="base_footprint_joint" type="fixed">
+    <origin xyz="0 0 0" rpy="0 0 0" />
+    <parent link="base_link" />
+    <child link="base_footprint" />
   </joint>
+  <gazebo reference="scanner">
+    <material>Gazebo/Blue</material>
+  </gazebo>
+  <!--gazebo>
+    <plugin filename="libgazebo_ros_diff_drive.so" name="differential_drive_controller">
+      <alwaysOn>true</alwaysOn>
+      <commandTopic>cmd_vel</commandTopic>
+      <leftJoint>base_to_lwheel_joint</leftJoint>
+      <legacyMode>false</legacyMode>
+      <odometryFrame>odom</odometryFrame>
+      <odometryTopic>odom</odometryTopic>
+      <publishOdomTF>true</publishOdomTF>
+      <publishWheelJointState>false</publishWheelJointState>
+      <publishWheelTF>true</publishWheelTF>
+      <rightJoint>base_to_rwheel_joint</rightJoint>
+      <robotBaseFrame>base_link</robotBaseFrame>
+      <rosDebugLevel>Debug</rosDebugLevel>
+      <torque>0.1</torque>
+      <updateRate>20</updateRate>
+      <wheelDiameter>${2*wheel_radius}</wheelDiameter>
+      <wheelSeparation>${body_width+(2*wheel_spacer)+wheel_width}</wheelSeparation>
+    </plugin>
+  </gazebo-->
   <!-- Parts -->
   <link name="base_link">
+    <collision>
+      <geometry>
+        <box size="${body_length} ${body_width} 0.0508"/>
+      </geometry>
+      <origin rpy="0 0 0" xyz="0 0 ${body_center_height}"/>
+    </collision>
     <visual>
       <geometry>
         <box size="${body_length} ${body_width} 0.0508"/>
       </geometry>
+      <material name="base" />
       <origin rpy="0 0 0" xyz="0 0 ${body_center_height}"/>
-      <material name="base" />
     </visual>
     <inertial>
@@ -53,129 +84,13 @@
     </inertial>
   </link>
-  <link name="lwheel">
-    <visual>
-      <geometry>
-        <cylinder length="${wheel_width}" radius="${wheel_radius}" />
-      </geometry>
-      <origin rpy="0 0 0" xyz="0 0 0"/>
-      <material name="wheel" />
-    </visual>
-    <inertial>
-        <origin xyz="0 0 0" rpy="0 0 0" />
-        <mass value="1" />
-        <inertia
-          ixx="1.0" ixy="0.0" ixz="0.0"
-          iyy="1.0" iyz="0.0"
-          izz="1.0" />
-    </inertial>
-    <collision name="lwheel_collision">
-      <geometry>
-        <cylinder length="${wheel_width}" radius="${wheel_radius}" />
-      </geometry>
-    </collision>
-  </link>
-  <joint name="base_to_lwheel" type="continuous">
-    <parent link="base_link"/>
-    <child link="lwheel"/>
-    <origin xyz="${wheel_forward_of_center_distance} ${(body_width/2)+wheel_spacer+(wheel_width/2)} ${wheel_width}" rpy="1.5708 0 0"/>
-    <axis xyz="0 0 1" />
-    <limit effort="0.0"  velocity="0.75" />
-  </joint>
-  <transmission name="left_wheel">
-    <type>transmission_interface/SimpleTransmission</type>
-    <joint name="base_to_lwheel">
-      <hardwareInterface>hardware_interface/VelocityJointInterface</hardwareInterface>
-    </joint>
-    <actuator name="left_motor">
-      <hardwareInterface>hardware_interface/VelocityJointInterface</hardwareInterface>
-      <mechanicalReduction>1</mechanicalReduction>
-    </actuator>
-  </transmission>
-  <link name="rwheel">
-    <visual>
-      <geometry>
-        <cylinder length="${wheel_width}" radius="${wheel_radius}" />
-      </geometry>
-      <origin rpy="0 0 0" xyz="0 0 0"/>
-      <material name="wheel" />
-    </visual>
-    <inertial>
-        <origin xyz="0 0 0" rpy="0 0 0" />
-        <mass value="1" />
-        <inertia
-          ixx="1.0" ixy="0.0" ixz="0.0"
-          iyy="1.0" iyz="0.0"
-          izz="1.0" />
-    </inertial>
-    <collision name="rwheel_collision">
-      <geometry>
-        <cylinder length="${wheel_width}" radius="${wheel_radius}" />
-      </geometry>
-    </collision>
-  </link>
-  <joint name="base_to_rwheel" type="continuous">
-    <parent link="base_link"/>
-    <child link="rwheel"/>
-    <origin xyz="${wheel_forward_of_center_distance} -${(body_width/2)+wheel_spacer+(wheel_width/2)} ${wheel_width}" rpy="-1.5708 0 0"/>
-    <axis xyz="0 0 1" />
-    <limit effort="0.0"  velocity="0.75" />
-  </joint>
-  <transmission name="right_wheel">
-    <type>transmission_interface/SimpleTransmission</type>
-    <joint name="base_to_rwheel">
-      <hardwareInterface>hardware_interface/VelocityJointInterface</hardwareInterface>
-    </joint>
-    <actuator name="right_motor">
-      <hardwareInterface>hardware_interface/VelocityJointInterface</hardwareInterface>
-      <mechanicalReduction>1</mechanicalReduction>
-    </actuator>
-  </transmission>
-  <link name="fwheel_attach">
-    <visual>
-      <geometry>
-        <cylinder length="0.060" radius="0.023"/>
-      </geometry>
-      <origin rpy="0 0 0" xyz="${fwheel_offset} 0 0.08"/>
-      <material name="white">
-        <color rgba="0.3 0.4 0.5 1"/>
-      </material>
-    </visual>
-    <inertial>
-        <origin xyz="0 0 0" rpy="0 0 0" />
-        <mass value="1" />
-        <inertia
-          ixx="1.0" ixy="0.0" ixz="0.0"
-          iyy="1.0" iyz="0.0"
-          izz="1.0" />
-    </inertial>
-  </link>
-  <joint name="base_to_fattach" type="fixed">
-    <parent link="base_link"/>
-    <child link="fwheel_attach"/>
-    <origin xyz="0 0 0" rpy="0 0 0"/>
-  </joint>
-  <link name="fwheel">
-    <visual>
-      <geometry>
-        <cylinder length="0.005" radius="0.020"/>
-      </geometry>
-      <origin rpy="1.578 0 0" xyz="0 0 0"/>
-      <material name="wheel" />
-    </visual>
-    <inertial>
-        <origin xyz="0 0 0" rpy="0 0 0" />
-        <mass value="1" />
-        <inertia
-          ixx="1.0" ixy="0.0" ixz="0.0"
-          iyy="1.0" iyz="0.0"
-          izz="1.0" />
-    </inertial>
-  </link>
-  <joint name="base_to_fwheel" type="continuous">
-    <parent link="base_link"/>
-    <child link="fwheel"/>
-    <origin xyz="${fwheel_offset} 0 0.02" rpy="0 0 0"/>
-    <axis xyz="0 0 1" />
-  </joint>
+  <xacro:wheel wheel_prefix="front_left" is_caster="false" >
+    <origin xyz="${wheel_forward_of_center_distance} ${(body_width/2)+wheel_spacer+(wheel_width/2)} ${wheel_radius}" rpy="0 0 0" />
+  </xacro:wheel>
+  <xacro:wheel wheel_prefix="front_right" is_caster="false" >
+    <origin xyz="${wheel_forward_of_center_distance} -${(body_width/2)+wheel_spacer+(wheel_width/2)} ${wheel_radius}" rpy="0 0 0" />
+  </xacro:wheel>
+  <xacro:wheel wheel_prefix="caster" is_caster="true" >
+    <origin xyz="${fwheel_offset} 0 ${wheel_radius}" rpy="0 0 0" />
+  </xacro:wheel>
   <link name="scanner">
     <visual>

Commit message: Temp sensor working, needs code. AMCL running. Pub odom with correct time.

File: motor_controller/urdf/lysander.xacro (robot description, xacro)
@@ -8,13 +8,13 @@
   <xacro:property name="wheel_forward_of_center_distance" value=".0762" />
   <xacro:property name="motor_height" value="0.0254" />
-  <xacro:property name="scanner_height" value="0.015" />
-  <xacro:property name="scanner_length" value="0.045" />
-  <xacro:property name="scanner_width" value="0.015" />
+  <xacro:property name="lidar_height" value="0.015" />
+  <xacro:property name="lidar_length" value="0.045" />
+  <xacro:property name="lidar_width" value="0.015" />
   <xacro:property name="wheel_radius" value="0.06" />
   <xacro:property name="wheel_spacer" value="0.00254" />
   <xacro:property name="wheel_width" value="0.060" />
   <xacro:property name="body_center_height" value="${wheel_radius+(motor_height/2)+(body_height/2)}" />
-  <xacro:property name="scanner_x_offset" value="${(body_length/2)-(scanner_width/2)}" />
-  <xacro:property name="scanner_z_offset" value="${body_center_height+(body_height/2)+(scanner_height/2)+.00508}" />
+  <xacro:property name="lidar_x_offset" value="${(body_length/2)-(lidar_width/2)}" />
+  <xacro:property name="lidar_z_offset" value="${body_center_height+(body_height/2)+(lidar_height/2)+.00508}" />
   <material name="base">
     <color rgba="0.25 0.25 0.53 1" />>
@@ -37,5 +37,5 @@
     <child link="base_footprint" />
   </joint>
-  <gazebo reference="scanner">
+  <gazebo reference="neato">
     <material>Gazebo/Blue</material>
   </gazebo>
@@ -93,14 +93,11 @@
     <origin xyz="${fwheel_offset} 0 ${wheel_radius}" rpy="0 0 0" />
   </xacro:wheel>
-  <link name="scanner">
-    <visual>
+  <link name="neato">
+    <collision>
       <geometry>
-        <box size="${scanner_width} ${scanner_length} ${scanner_height}"/>
+        <box size="${lidar_width} ${lidar_length} ${lidar_height}"/>
       </geometry>
       <origin rpy="0 0 0" xyz="0 0 0"/>
-      <material name="black">
-        <color rgba="0.5 0 0 1"/>
-      </material>
-    </visual>
+    </collision>
     <inertial>
         <origin xyz="0 0 0" rpy="0 0 0" />
@@ -111,9 +108,18 @@
           izz="1.0" />
     </inertial>
+    <visual>
+      <geometry>
+        <box size="${lidar_width} ${lidar_length} ${lidar_height}"/>
+      </geometry>
+      <origin rpy="0 0 0" xyz="0 0 0"/>
+      <material name="black">
+        <color rgba="0.5 0 0 1"/>
+      </material>
+    </visual>
   </link>
-  <joint name="base_to_scanner" type="fixed">
+  <joint name="base_to_neato" type="fixed">
     <parent link="base_link"/>
-    <child link="scanner"/>
-    <origin xyz="${scanner_x_offset} 0  ${scanner_z_offset}" rpy="0 0 0"/>
+    <child link="neato"/>
+    <origin xyz="${lidar_x_offset} 0  ${lidar_z_offset}" rpy="0 0 0"/>
   </joint>
 </robot>
